File: eagle/808_rs.brd (EAGLE design)
At the start: 100 x 80 mm, 75 parts, among them IC1 TL072P, IC2 TL072P, Q1 2SK30, Q59 2N3904, Q60 2N3906, Q61 2N3904, Q62 2N3904, Q63 2N3904, SW8 808_LT_MSS42_SW_4PDT

Commit message: 93pct auto
Parts:
- R305, R306, R310, R311, R316, R323, R324, R325, R326, R331: device TR808clone:0207/5V -> TR808clone:0207/7
- R313: device TR808clone:0207/5V -> TR808clone:0309/12
- R318: device TR808clone:0207/5V -> TR808clone:0207/2V
- moved R313 15.3 mm to (73.7, 53.3), turned to 90 degrees
- moved R321 10.5 mm to (31.8, 27.9)
- moved R310 10.2 mm to (40.6, 38.1), turned to 180 degrees
- moved R108 9.92 mm to (25.4, 33.0)
- moved C120 9.25 mm to (40.6, 27.9), turned to 270 degrees
- moved D63 9.16 mm to (26.7, 30.5)
- moved C121 8.98 mm to (34.3, 33.0), turned to 90 degrees
- moved C112 7.41 mm to (25.4, 16.5)
- moved R304 7.41 mm to (27.9, 25.4)
- moved R238 6.84 mm to (71.1, 17.8), turned to 90 degrees
- moved R322 6.84 mm to (41.9, 44.5)
- moved R107 6.84 mm to (29.2, 40.6)
- moved C122 6.48 mm to (38.1, 43.2)
- moved R300 6.35 mm to (25.4, 49.5)
- moved TRIGGER 6.35 mm to (12.7, 59.7)
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Routing:
- net GND: track 0.00 -> 346.2 mm
- net N$338: track 0.00 -> 120.2 mm
- net N$8: track 0.00 -> 108.3 mm
- net +12V: track 0.00 -> 101.4 mm
- net N$351: track 0.00 -> 87.8 mm
- net N$6: track 0.00 -> 66.7 mm
- net N$348: track 0.00 -> 50.0 mm
- net N$357: track 0.00 -> 44.0 mm
- net N$355: track 0.00 -> 43.7 mm
- net TRIG: track 0.00 -> 42.8 mm
- net RS: track 0.00 -> 35.3 mm
- net N$161: track 0.00 -> 31.1 mm
- net N$344: track 0.00 -> 30.7 mm
- net -12V: track 0.00 -> 28.9 mm
- net N$165: track 0.00 -> 28.6 mm
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