File: eagle/808_rs.sch (EAGLE design)
At the start: 75 parts, among them IC1 TL072P, IC2 TL072P, Q1 2SK30, Q59 2N3904, Q60 2N3906, Q61 2N3904, Q62 2N3904, Q63 2N3904, SW8 808_LT_MSS42_SW_4PDT

Commit message: routed
Parts:
- C1: device TR808clone:C-EU025-025X050 -> TR808clone:C-EU050-024X044
- C112, C118: device TR808clone:C-EU050-024X044 -> TR808clone:C-EU050-025X075
- C113: device TR808clone:C-EU075-032X103 -> TR808clone:C-EU050-025X075
- C117, C119: device TR808clone:C-EU3.5MM_PITCH -> TR808clone:C-EU050-024X044
- C120: device TR808clone:CPOL-EUE2.5-5 -> TR808clone:CPOL-EUE2.5-6
- C125: device TR808clone:C-EU3.5MM_PITCH -> TR808clone:C-EU050-025X075
- R312, R314, R318: device TR808clone:R-EU_0207/5V -> TR808clone:R-EU_0207/7
- R331: device TR808clone:R-EU_0207/7 -> TR808clone:R-EU_0207/5V
Changed lines of the file:
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@@
 <part name="V210" library="supply1" deviceset="GND" device=""/>
 <part name="R308" library="TR808clone" deviceset="R-EU_" device="0207/5V" value="820K"/>
-<part name="C119" library="TR808clone" deviceset="C-EU" device="3.5MM_PITCH" value="2.2n"/>
-<part name="C117" library="TR808clone" deviceset="C-EU" device="3.5MM_PITCH" value="2.2n"/>
-<part name="C118" library="TR808clone" deviceset="C-EU" device="050-024X044" value="2.2n"/>
-<part name="R312" library="TR808clone" deviceset="R-EU_" device="0207/5V" value="1K"/>
+<part name="C119" library="TR808clone" deviceset="C-EU" device="050-024X044" value="2.2n"/>
+<part name="C117" library="TR808clone" deviceset="C-EU" device="050-024X044" value="2.2n"/>
+<part name="C118" library="TR808clone" deviceset="C-EU" device="050-025X075" value="2.2n"/>
+<part name="R312" library="TR808clone" deviceset="R-EU_" device="0207/7" value="1K"/>
 <part name="V211" library="supply1" deviceset="GND" device=""/>
-<part name="R314" library="TR808clone" deviceset="R-EU_" device="0207/5V" value="33K"/>
+<part name="R314" library="TR808clone" deviceset="R-EU_" device="0207/7" value="33K"/>
 <part name="R313" library="TR808clone" deviceset="R-EU_" device="0309/12" value="390K"/>
 <part name="V212" library="supply1" deviceset="GND" device=""/>
 <part name="R309" library="TR808clone" deviceset="R-EU_" device="0207/2V" value="33K"/>
 <part name="R319" library="TR808clone" deviceset="R-EU_" device="0207/5V" value="220K"/>
-<part name="C125" library="TR808clone" deviceset="C-EU" device="3.5MM_PITCH" value="10n"/>
+<part name="C125" library="TR808clone" deviceset="C-EU" device="050-025X075" value="10n"/>
 <part name="R326" library="TR808clone" deviceset="R-EU_" device="0309/10" value="10K"/>
-<part name="R331" library="TR808clone" deviceset="R-EU_" device="0207/7" value="47K"/>
+<part name="R331" library="TR808clone" deviceset="R-EU_" device="0207/5V" value="47K"/>
 <part name="V213" library="supply1" deviceset="GND" device=""/>
 <part name="C153" library="TR808clone" deviceset="C-EU" device="025-025X050" value="22p"/>
@@
 <part name="V214" library="supply1" deviceset="GND" device=""/>
 <part name="R316" library="TR808clone" deviceset="R-EU_" device="0207/5V" value="1M"/>
-<part name="R318" library="TR808clone" deviceset="R-EU_" device="0207/5V" value="220K"/>
+<part name="R318" library="TR808clone" deviceset="R-EU_" device="0207/7" value="220K"/>
 <part name="R317" library="TR808clone" deviceset="R-EU_" device="0207/5V" value="10K"/>
 <part name="Q62" library="808_lt" deviceset="2N3904" device=""/>
 <part name="V215" library="supply1" deviceset="GND" device=""/>
 <part name="R321" library="TR808clone" deviceset="R-EU_" device="0207/7" value="2M2"/>
-<part name="C120" library="TR808clone" deviceset="CPOL-EU" device="E2.5-5" value="10/16"/>
+<part name="C120" library="TR808clone" deviceset="CPOL-EU" device="E2.5-6" value="10/16"/>
 <part name="V217" library="supply1" deviceset="GND" device=""/>
 <part name="R300" library="TR808clone" deviceset="R-EU_" device="0207/5V" value="22K"/>
@@
 <part name="R320" library="TR808clone" deviceset="R-EU_" device="0207/7" value="22K"/>
 <part name="Q61" library="808_lt" deviceset="2N3904" device=""/>
-<part name="C112" library="TR808clone" deviceset="C-EU" device="050-024X044" value="22n"/>
-<part name="C113" library="TR808clone" deviceset="C-EU" device="075-032X103" value="47n"/>
+<part name="C112" library="TR808clone" deviceset="C-EU" device="050-025X075" value="22n"/>
+<part name="C113" library="TR808clone" deviceset="C-EU" device="050-025X075" value="47n"/>
 <part name="R304" library="TR808clone" deviceset="R-EU_" device="0207/5V" value="47K"/>
 <part name="R305" library="TR808clone" deviceset="R-EU_" device="0207/7" value="1M"/>
@@
 <part name="V2" library="supply1" deviceset="GND" device=""/>
 <part name="V3" library="supply1" deviceset="GND" device=""/>
-<part name="C1" library="TR808clone" deviceset="C-EU" device="025-025X050" value="22p"/>
+<part name="C1" library="TR808clone" deviceset="C-EU" device="050-024X044" value="22p"/>
 <part name="C2" library="TR808clone" deviceset="C-EU" device="025-025X050" value="22p"/>
 <part name="C3" library="TR808clone" deviceset="C-EU" device="025-025X050" value="22p"/>

Commit message: almost rerouted
Parts:
- C2, C3: device TR808clone:C-EU025-025X050 -> TR808clone:C-EU050-024X044
- R312, R320, R323: device TR808clone:R-EU_0207/7 -> TR808clone:R-EU_0207/5V
- R324: device TR808clone:R-EU_0207/7 -> TR808clone:R-EU_0309/10
- R331: device TR808clone:R-EU_0207/5V -> TR808clone:R-EU_0207/7
Changed lines of the file:
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@@
 <part name="R325" library="TR808clone" deviceset="R-EU_" device="0207/7" value="330K"/>
 <part name="Q63" library="808_lt" deviceset="2N3904" device=""/>
-<part name="R323" library="TR808clone" deviceset="R-EU_" device="0207/7" value="22K"/>
+<part name="R323" library="TR808clone" deviceset="R-EU_" device="0207/5V" value="22K"/>
 <part name="R322" library="TR808clone" deviceset="R-EU_" device="0207/7" value="10K"/>
 <part name="V204" library="supply1" deviceset="GND" device=""/>
@@
 <part name="C117" library="TR808clone" deviceset="C-EU" device="050-024X044" value="2.2n"/>
 <part name="C118" library="TR808clone" deviceset="C-EU" device="050-025X075" value="2.2n"/>
-<part name="R312" library="TR808clone" deviceset="R-EU_" device="0207/7" value="1K"/>
+<part name="R312" library="TR808clone" deviceset="R-EU_" device="0207/5V" value="1K"/>
 <part name="V211" library="supply1" deviceset="GND" device=""/>
 <part name="R314" library="TR808clone" deviceset="R-EU_" device="0207/7" value="33K"/>
@@
 <part name="C125" library="TR808clone" deviceset="C-EU" device="050-025X075" value="10n"/>
 <part name="R326" library="TR808clone" deviceset="R-EU_" device="0309/10" value="10K"/>
-<part name="R331" library="TR808clone" deviceset="R-EU_" device="0207/5V" value="47K"/>
+<part name="R331" library="TR808clone" deviceset="R-EU_" device="0207/7" value="47K"/>
 <part name="V213" library="supply1" deviceset="GND" device=""/>
 <part name="C153" library="TR808clone" deviceset="C-EU" device="025-025X050" value="22p"/>
@@
 <part name="R300" library="TR808clone" deviceset="R-EU_" device="0207/5V" value="22K"/>
 <part name="VR16" library="pot" deviceset="3RP/1610N" device="" value="100KA"/>
-<part name="R324" library="TR808clone" deviceset="R-EU_" device="0207/7" value="220K"/>
-<part name="R320" library="TR808clone" deviceset="R-EU_" device="0207/7" value="22K"/>
+<part name="R324" library="TR808clone" deviceset="R-EU_" device="0309/10" value="220K"/>
+<part name="R320" library="TR808clone" deviceset="R-EU_" device="0207/5V" value="22K"/>
 <part name="Q61" library="808_lt" deviceset="2N3904" device=""/>
 <part name="C112" library="TR808clone" deviceset="C-EU" device="050-025X075" value="22n"/>
@@
 <part name="V3" library="supply1" deviceset="GND" device=""/>
 <part name="C1" library="TR808clone" deviceset="C-EU" device="050-024X044" value="22p"/>
-<part name="C2" library="TR808clone" deviceset="C-EU" device="025-025X050" value="22p"/>
-<part name="C3" library="TR808clone" deviceset="C-EU" device="025-025X050" value="22p"/>
+<part name="C2" library="TR808clone" deviceset="C-EU" device="050-024X044" value="22p"/>
+<part name="C3" library="TR808clone" deviceset="C-EU" device="050-024X044" value="22p"/>
 <part name="C4" library="TR808clone" deviceset="C-EU" device="050-024X044" value="22p"/>
 <part name="TRIGGER" library="solpad" deviceset="LSP11" device=""/>
