File: eagle/808_rs.sch (EAGLE design)
At the start: 75 parts, among them IC1 TL072P, IC2 TL072P, Q1 2SK30, Q59 2N3904, Q60 2N3906, Q61 2N3904, Q62 2N3904, Q63 2N3904, SW8 808_LT_MSS42_SW_4PDT

Commit message: rerouted
Parts:
- R320: device TR808clone:R-EU_0207/5V -> TR808clone:R-EU_0207/7
Changed lines of the file:
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@@
 <part name="VR16" library="pot" deviceset="3RP/1610N" device="" value="100KA"/>
 <part name="R324" library="TR808clone" deviceset="R-EU_" device="0309/10" value="220K"/>
-<part name="R320" library="TR808clone" deviceset="R-EU_" device="0207/5V" value="22K"/>
+<part name="R320" library="TR808clone" deviceset="R-EU_" device="0207/7" value="22K"/>
 <part name="Q61" library="808_lt" deviceset="2N3904" device=""/>
 <part name="C112" library="TR808clone" deviceset="C-EU" device="050-025X075" value="22n"/>

Commit message: tweaks
Parts:
- R305, R318: device TR808clone:R-EU_0207/7 -> TR808clone:R-EU_0207/5V
- R313: device TR808clone:R-EU_0309/12 -> TR808clone:R-EU_0207/7
- R316: device TR808clone:R-EU_0207/5V -> TR808clone:R-EU_0207/2V
- R324: device TR808clone:R-EU_0309/10 -> TR808clone:R-EU_0207/7
Changed lines of the file:
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@@
 <part name="V211" library="supply1" deviceset="GND" device=""/>
 <part name="R314" library="TR808clone" deviceset="R-EU_" device="0207/7" value="33K"/>
-<part name="R313" library="TR808clone" deviceset="R-EU_" device="0309/12" value="390K"/>
+<part name="R313" library="TR808clone" deviceset="R-EU_" device="0207/7" value="390K"/>
 <part name="V212" library="supply1" deviceset="GND" device=""/>
 <part name="R309" library="TR808clone" deviceset="R-EU_" device="0207/2V" value="33K"/>
@@
 <part name="R315" library="TR808clone" deviceset="R-EU_" device="0207/5V" value="5K6"/>
 <part name="V214" library="supply1" deviceset="GND" device=""/>
-<part name="R316" library="TR808clone" deviceset="R-EU_" device="0207/5V" value="1M"/>
-<part name="R318" library="TR808clone" deviceset="R-EU_" device="0207/7" value="220K"/>
+<part name="R316" library="TR808clone" deviceset="R-EU_" device="0207/2V" value="1M"/>
+<part name="R318" library="TR808clone" deviceset="R-EU_" device="0207/5V" value="220K"/>
 <part name="R317" library="TR808clone" deviceset="R-EU_" device="0207/5V" value="10K"/>
 <part name="Q62" library="808_lt" deviceset="2N3904" device=""/>
@@
 <part name="R300" library="TR808clone" deviceset="R-EU_" device="0207/5V" value="22K"/>
 <part name="VR16" library="pot" deviceset="3RP/1610N" device="" value="100KA"/>
-<part name="R324" library="TR808clone" deviceset="R-EU_" device="0309/10" value="220K"/>
+<part name="R324" library="TR808clone" deviceset="R-EU_" device="0207/7" value="220K"/>
 <part name="R320" library="TR808clone" deviceset="R-EU_" device="0207/7" value="22K"/>
 <part name="Q61" library="808_lt" deviceset="2N3904" device=""/>
@@
 <part name="C113" library="TR808clone" deviceset="C-EU" device="050-025X075" value="47n"/>
 <part name="R304" library="TR808clone" deviceset="R-EU_" device="0207/5V" value="47K"/>
-<part name="R305" library="TR808clone" deviceset="R-EU_" device="0207/7" value="1M"/>
+<part name="R305" library="TR808clone" deviceset="R-EU_" device="0207/5V" value="1M"/>
 <part name="V409" library="supply1" deviceset="GND" device=""/>
 <part name="R327" library="TR808clone" deviceset="R-EU_" device="0207/5V" value="470K"/>
